File: FireflyV0.kicad_pcb (KiCad board)
At the start: 2 copper layers, 64.2 x 43.3 mm, 15 parts, among them IC1 MXC6655XA, J1 USB4125-GF-A-0190, J2 USB4125-GF-A-0190, U1 Pico, U2 LEDS4, U3 LEDS4, U4 LEDS4, U5 LEDS4

Commit message: Uploading ordered rev1 files
Parts:
- added R1: R_US, Resistor_SMD:R_0805_2012Metric, F.Cu at (68.4, 46.5)
- added R2: R_US, Resistor_SMD:R_0805_2012Metric, F.Cu at (70.3, 46.5)
- added R3: R_US, Resistor_SMD:R_0805_2012Metric, F.Cu at (18.1, 46.3)
- added R4: R_US, Resistor_SMD:R_0805_2012Metric, F.Cu at (20.1, 46.3)
- C1: footprint Capacitor_SMD:C_0805_2012Metric -> SamacSys_Parts:CAPC2012X88N
- moved C1 0.16 mm to (64.5, 43.5), turned to 90 degrees
Connections:
- C1 pad 1: GND -> 3V3
- C1 pad 2: 3V3 -> GND
- J1 pad A5: unconnected-(J1-PadA5) -> Net-(J1-PadA5)
- J1 pad B5: unconnected-(J1-PadB5) -> Net-(J1-PadB5)
- J2 pad A5: unconnected-(J2-PadA5) -> Net-(J2-PadA5)
- J2 pad B5: unconnected-(J2-PadB5) -> Net-(J2-PadB5)
Routing:
- net GND: track 104.2 -> 113.1 mm
- net Net-(J1-PadA5): track 0.00 -> 4.00 mm
- net Net-(J1-PadB5): track 0.00 -> 3.42 mm
- net Net-(J2-PadA5): track 0.00 -> 3.21 mm
- net Net-(J2-PadB5): track 0.00 -> 2.77 mm
- net ACC_INT: track 35.7 -> 34.7 mm, vias 2 -> 1
- net ACC_CLK: track 33.6 -> 34.0 mm, vias 2 -> 1
- net ACC_DATA: track 30.5 -> 30.3 mm, vias 2 -> 1
Other:
- board text added: "6/29/2022"
- board text added: "@KylarLEDs FireFlyV1"
- board text added: "ACLK"
- board text added: "ADAT"
- board text added: "AINT"
- board text added: "BTN1"
- board text added: "BTN2"
- board text added: "POT1"
- board text added: "POT2"
- board text added: "acc_clk =gp7 acc_data=gp6 acc_int =gp5 pdm_clk =gp21 pdm_data=gp20"
- board text added: "clk_3 =gp11 data_3=gp10 clk_4 =gp13 data_4=gp12"
- board text added: "pot_1 =gp27 pot_2 =gp26 btn_1 =gp9 btn_2 =gp8"
- board text removed: "4/25/2022"
- board text removed: "@KylarLEDs FireFlyV0"
- board text removed: "POT_ADC"
- board text removed: "led1 =gp16 led2 =gp17 apa =gp15"
- board text removed: "pot_1 =gp27 pot_2 =gp26"
