File: CircleBoard/CircleBoard.kicad_pcb (KiCad board)
At the start: 2 copper layers, 265.8 x 268.2 mm, 110 parts, among them J1 USB4125-GF-A-0190, U1 Pico

Commit message: CircleBoard updates
Parts:
- removed RV1, RV2: R_Potentiometer, Varistor:3352T-1-104LF
- added VR1: PTV09A-2020F-A104, SamacSys_Parts:PTV09A2020FA104, F.Cu at (128.6, -4.94)
- added VR2: PTV09A-2020F-A104, SamacSys_Parts:PTV09A2020FA104, F.Cu at (141.1, -4.96)
- added led100: LED_WS2812B_PLCC4_5.0x5.0mm_P3.2mm, LED_WS2812B_PLCC4_5.0x5.0mm_P3.2mm, F.Cu at (94.7, 248.4)
- added led101: LED_WS2812B_PLCC4_5.0x5.0mm_P3.2mm, LED_WS2812B_PLCC4_5.0x5.0mm_P3.2mm, F.Cu at (160.9, 248.3)
- S1, S2: value EVQ-9P701P -> 1-1825027-7; footprint SamacSys_Parts:EVQ-9P701P -> SamacSys_Parts:118250277
- XD1, XD2: renamed from ?; value (none) -> MountingHole_3.2mm_M3_DIN965_Pad; footprint (none) -> MountingHole:MountingHole_3.2mm_M3_DIN965_Pad
- moved led34 209.7 mm to (38.2, 91.8)
- moved led27 198.0 mm to (218.1, 92.5)
- moved led85 186.8 mm to (220.6, 196.2)
- moved led86 178.7 mm to (216.8, 215.8)
- moved led40 178.1 mm to (242.8, 113.4)
- moved led61 175.5 mm to (65.5, 144.3)
- moved led48 170.1 mm to (32.8, 111.3)
- moved led28 157.3 mm to (193.8, 89.2)
- moved led33 155.0 mm to (62.0, 89.7)
- moved led47 154.8 mm to (86.7, 116.0)
- moved led26 152.8 mm to (233.6, 81.5)
- moved led84 138.3 mm to (203.3, 187.6)
- moved led41 138.1 mm to (223.6, 113.0)
- moved led90 136.4 mm to (59.2, 219.3)
- moved led35 136.3 mm to (21.2, 81.9)
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Connections:
- S1 pad 1: GND -> BTN_1
- S1 pad 2: BTN_1 -> GND
- S2 pad 1: GND -> BTN_2
- S2 pad 2: BTN_2 -> GND
- led0 pad 4: LED_DATA_1 -> LINK00
Routing:
- net LINK101: track 0.00 -> 74.8 mm, vias 0 -> 2
- net LED_DATA_1: track 69.4 -> 0.00 mm, vias 2 -> 0
- net LINK35: track 86.7 -> 19.4 mm, vias 2 -> 0
- net GND: track 26.3 -> 92.6 mm, vias 108 -> 112
- net LINK26: track 88.0 -> 22.1 mm, vias 2 -> 0
- net LINK40: track 40.8 -> 103.2 mm, vias 0 -> 2
- net LINK62: track 89.2 -> 30.5 mm, vias 2 -> 0
- net LINK64: track 93.2 -> 35.8 mm, vias 2 -> 0
- net 3V3: track 68.1 -> 121.2 mm, vias 2 -> 1
- net LINK39: track 26.3 -> 74.3 mm, vias 0 -> 2
- net LINK36: track 60.7 -> 15.6 mm, vias 2 -> 0
- net LINK73: track 58.9 -> 14.1 mm, vias 2 -> 0
- net LINK27: track 57.6 -> 13.8 mm, vias 2 -> 0
- net PDM_CLK: track 24.3 -> 67.6 mm
- net LINK49: track 58.1 -> 15.1 mm, vias 2 -> 0
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Other:
- board size 265.8 x 268.2 mm -> 266.5 x 270.4 mm
