File: FireFlyV1.1/FireFlyV1.kicad_pcb (KiCad board)
At the start: 2 copper layers, 64 x 26.2 mm, 59 parts, among them J1 Conn_01x03, J2 Conn_01x01_Pin, J3 Conn_01x01_Pin, SW1 TS-1187A-B-A-B, SW2 TS-1187A-B-A-B, U1 RP2040, U2 W25Q32JVSS, U3 AMS1117-3.3, U5 MCP6001T-I/OT, U7 PEC12R-4215F-S0024, X1 X322512MSB4SI

Commit message: Questionable routing decisions
Parts:
- moved C3 1.73 mm to (210.6, 112.5)
- moved C15 0.99 mm to (212.6, 112.7)
- moved C2 0.90 mm to (214.4, 113.1)
- moved X1 0.61 mm to (220.6, 115.9)
- moved R24 0.43 mm to (233.9, 104.0)
- moved R25 0.43 mm to (231.8, 103.8)
- moved C9 0.21 mm to (233.9, 105.0)
- moved C10 0.16 mm to (231.8, 104.9)
Routing:
- net +5V: track 78.6 -> 0.00 mm, vias 3 -> 0
- net 3V3: track 71.1 -> 0.00 mm, vias 2 -> 0
- net Net-(SW2-D): track 19.6 -> 0.00 mm, vias 2 -> 0
- net Net-(U5-VIN-): track 18.5 -> 0.00 mm, vias 2 -> 0
- net Net-(U1-VREG_VOUT): track 12.6 -> 0.00 mm, vias 2 -> 0
- net MIC_ADC: track 12.3 -> 0.00 mm
- net Net-(U5-VIN+): track 12.0 -> 0.00 mm
- net XIN: track 11.2 -> 0.00 mm, vias 2 -> 0
- net /B: track 10.3 -> 0.00 mm
- net Net-(X1-OSC2): track 9.19 -> 0.00 mm
- net MIC_RAW_OUT: track 8.66 -> 0.00 mm
- net Net-(USB1-CC2): track 6.61 -> 0.00 mm
- net USB_DP: track 6.58 -> 0.00 mm
- net Net-(USB1-CC1): track 6.45 -> 0.00 mm
- net Net-(R15-Pad1): track 6.04 -> 0.00 mm
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Other:
- board size 64 x 26.2 mm -> 64 x 27.7 mm
