File: FireFlyV3_0/FireFlyV3_0.kicad_pcb (KiCad board)
At the start: 4 copper layers, 75 x 22 mm, 61 parts, among them J1 Conn_01x23, J2 Conn_01x23, SW1 BTN, SW2 BTN, SW3 BTN, SW4 BTN, U2 W25Q128JVS, U3 RP2040, U4 AMS1117-3.3, U5 ESP32-C3FH4, Y1 12MHz, X322512MSB4SI, Y2 40MHz, X252040MMB4SI

Commit message: Added V1_3 and V3_1.
Other:
- board text added: "FireFlyV3.1 @KylarLEDs 02-02-2025"
- board text added: "i love jlcpcb"
- board text removed: "FireFlyV3.0 @KylarLEDs 12-1-2024"
Changed lines of the file:
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@@
 		)
 	)
-	(gr_text "FireFlyV3.0\n@KylarLEDs\n12-1-2024"
+	(gr_text "FireFlyV3.1\n@KylarLEDs\n02-02-2025"
 		(at 173.515 87.88 0)
 		(layer "B.SilkS")
 		(effects
+			(font
+				(size 3 3)
+				(thickness 0.5)
+				(bold yes)
+			)
+			(justify left bottom mirror)
+		)
+	)
+	(gr_text "i love jlcpcb"
+		(at 140.815 83.18 0)
+		(layer "B.SilkS")
+		(effects
